Commit message: Rename of sim demo pkg

File: panther_sim_demo/urdf/panther.urdf (robot description, URDF)
Before this commit: robot lexus_rx_450h, 6 links, 5 joints
Links:
- link base_link: geometry collision box size=5.5 2.25 2; visual mesh filename=package://panther_sim_demo/meshes/Panther_v1.0.stl scale=0.001 0.001 0.001
