Commit message: Panther changes

File: panther_real_demo/urdf/panther.urdf (robot description, URDF)
Before this commit: robot lexus_rx_450h, 6 links, 5 joints
Links:
- removed link lidar_front
- removed link lidar_rear
- added link os_sensor, mass 0.1; collision cylinder length=0.0869 radius=0.05165; visual cylinder length=0.0869 radius=0.05165
Joints:
- removed joint lidar_front_joint
- removed joint lidar_rear_joint
- added joint os_sensor_joint: type fixed, parent base_link, child os_sensor, origin xyz=0.42 0.0 0.19 rpy=0 0 0
