Commit message: Panther simulation demo parameters tuned

File: adehome/AutowareDemo/src/panther_description/urdf/panther.urdf (robot description, URDF)
Before this commit: robot panther, 5 links, 4 joints
Links:
- link base_link: geometry collision box size=5.5 2.25 2; visual mesh filename=package://panther_description/meshes/Panther_v1.0.stl scale=0.001 0.001 0.001
